File: sahaischedule.kicad_pcb (KiCad board)
At the start: 2 copper layers, 32.4 x 49 mm, 48 parts, among them J1 USB_B_Micro, J2 SSD1306, J3 SSD1306, J4 SSD1306, J5 SSD1306, J6 JTAG/SWD, Q1 SUD08P06-155L, SW1 Butt, SW2 Butt, SW3 Butt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

Commit message: added my name
Other:
- board text added: "Sahai Timer Copyleft Elam Day-Friedland 2021"
Changed lines of the file:
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@@
   )
   (gr_rect (start 163.322 76.454) (end 130.937 125.476) (layer "Edge.Cuts") (width 0.2) (fill none))
+  (gr_text "Sahai Timer\nCopyleft Elam Day-Friedland 2021" (at 141.6304 123.7488) (layer "F.SilkS")
+    (effects (font (size 0.75 0.75) (thickness 0.15)))
+  )
   (segment (start 138.483187 107.67825) (end 137.29725 107.67825) (width 0.25) (layer "F.Cu") (net 1))
   (segment (start 138.85 86.9672) (end 140.4366 88.5538) (width 0.25) (layer "F.Cu") (net 1))
